File: ATS.kicad_sch (KiCad schematic)
At the start: 10 parts

Commit message: incorporated libraries
Parts:
- TEENSY4.1_1: symbol DEV-16771:DEV-16771 -> Teensy4.1:DEV-16771
Changed lines of the file:
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@@
 	)
 	(symbol
-		(lib_id "DEV-16771:DEV-16771")
+		(lib_id "Teensy4.1:DEV-16771")
 		(at 110.49 101.6 0)
 		(unit 1)
